File: rfm98pw-wing.sch (EAGLE design)
At the start: 14 parts, among them X4 uFL

Commit message: Images and license
Parts:
- renumbered U$11 to R1
Other:
- note removed: "BREAKOUTS"
Changed lines of the file:
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@@
 <attributes>
 <attribute name="PROJECT_AUTHOR" value="Tinkerman &lt;xose.perez@gmail.com&gt;"/>
-<attribute name="PROJECT_LICENSE" value="CC-SA-BY-NC 4.0 Intl."/>
+<attribute name="PROJECT_LICENSE" value="CC-BY-SA 4.0 Intl."/>
 <attribute name="PROJECT_NAME" value="RFM98PW Feather Wing"/>
 <attribute name="PROJECT_VERSION" value="0.1.20190707"/>
@@
 <part name="X4" library="adafruit" deviceset="ANTENNA_U.FL" device="" value="uFL"/>
 <part name="U$24" library="xose" deviceset="RFM95PW-RFM98PW" device=""/>
-<part name="FRAME1" library="xose" deviceset="DINA4_L" device="">
-<attribute name="PROJECT_AUTHOR" value=""/>
-<attribute name="PROJECT_LICENSE" value=""/>
-<attribute name="PROJECT_NAME" value=""/>
-<attribute name="PROJECT_VERSION" value=""/>
-</part>
 <part name="X1" library="adafruit" deviceset="SMACONNECTOR" device="_EDGE"/>
 <part name="U$1" library="microbuilder" deviceset="GND" device=""/>
@@
 <part name="D1" library="xose" deviceset="DIODE" device="-SMD"/>
 <part name="D0" library="xose" deviceset="DIODE" device="-SMD"/>
-<part name="U$11" library="xose" deviceset="RESISTOR" device="0805" value="10K"/>
+<part name="R1" library="xose" deviceset="RESISTOR" device="0805" value="10K"/>
 <part name="U$16" library="microbuilder" deviceset="GND" device=""/>
 <part name="U$21" library="microbuilder" deviceset="GND" device=""/>
 <part name="U$7" library="microbuilder" deviceset="GND" device=""/>
 <part name="L1" library="Spark" deviceset="INDUCTOR-SPARKFUN" device="0805"/>
+<part name="FRAME1" library="xose" deviceset="DINA4_L" device=""/>
 </parts>
 <sheets>
 <sheet>
 <plain>
-<text x="172.72" y="83.82" size="1.778" layer="94">BREAKOUTS</text>
 </plain>
 <instances>
@@
 </instance>
 <instance part="JP1" gate="A" x="226.06" y="101.6" smashed="yes" rot="R180">
-<attribute name="NAME" x="232.41" y="80.645" size="1.778" layer="95" rot="R180"/>
 <attribute name="VALUE" x="232.41" y="127" size="1.778" layer="96" rot="R180"/>
 </instance>
@@
 </instance>
 <instance part="JP3" gate="G$1" x="195.58" y="106.68" smashed="yes">
-<attribute name="NAME" x="189.23" y="125.095" size="1.778" layer="95"/>
 <attribute name="VALUE" x="189.23" y="88.9" size="1.778" layer="96"/>
 </instance>
@@
 </instance>
 <instance part="U$24" gate="G$1" x="68.58" y="121.92" smashed="yes"/>
-<instance part="FRAME1" gate="G$1" x="0" y="0" smashed="yes"/>
-<instance part="FRAME1" gate="G$2" x="162.56" y="0" smashed="yes">
-<attribute name="PROJECT_NAME" x="180.34" y="22.86" size="2.54" layer="94"/>
-<attribute name="PROJECT_AUTHOR" x="180.34" y="15.24" size="2.54" layer="94"/>
-<attribute name="PROJECT_VERSION" x="180.34" y="2.54" size="2.54" layer="94"/>
-<attribute name="PROJECT_LICENSE" x="180.34" y="10.16" size="2.54" layer="94"/>
-</instance>
 <instance part="X1" gate="G$1" x="99.06" y="66.04" smashed="yes">
 <attribute name="NAME" x="106.68" y="68.58" size="1.27" layer="95"/>
@@
 <attribute name="NAME" x="101.6" y="109.22" size="0.8128" layer="95" font="vector" ratio="15" align="bottom-center"/>
 </instance>
-<instance part="U$11" gate="G$1" x="116.84" y="106.68" smashed="yes" rot="R90">
+<instance part="R1" gate="G$1" x="116.84" y="106.68" smashed="yes" rot="R90">
 <attribute name="NAME" x="115.57" y="106.68" size="0.8128" layer="94" font="vector" ratio="15" rot="R90" align="bottom-center"/>
 <attribute name="VALUE" x="118.11" y="106.68" size="0.8128" layer="94" font="vector" ratio="15" rot="R90" align="top-center"/>
@@
 <attribute name="NAME" x="38.1" y="68.58" size="1.778" layer="95" rot="R90"/>
 <attribute name="VALUE" x="48.26" y="68.58" size="1.778" layer="96" rot="R90"/>
+</instance>
+<instance part="FRAME1" gate="G$1" x="0" y="0" smashed="yes"/>
+<instance part="FRAME1" gate="G$2" x="162.56" y="0" smashed="yes">
+<attribute name="PROJECT_VERSION" x="180.34" y="2.54" size="2.54" layer="94"/>
+<attribute name="PROJECT_NAME" x="180.34" y="22.86" size="2.54" layer="94"/>
+<attribute name="PROJECT_LICENSE" x="180.34" y="10.16" size="2.54" layer="94"/>
+<attribute name="PROJECT_AUTHOR" x="180.34" y="15.24" size="2.54" layer="94"/>
 </instance>
 </instances>
@@
 </segment>
 <segment>
-<pinref part="U$11" gate="G$1" pin="1"/>
+<pinref part="R1" gate="G$1" pin="1"/>
 <pinref part="U$16" gate="G$1" pin="GND"/>
 <wire x1="116.84" y1="101.6" x2="116.84" y2="99.06" width="0.1524" layer="91"/>
@@
 <wire x1="104.14" y1="111.76" x2="111.76" y2="111.76" width="0.1524" layer="91"/>
 <wire x1="111.76" y1="111.76" x2="111.76" y2="114.3" width="0.1524" layer="91"/>
-<pinref part="U$11" gate="G$1" pin="2"/>
+<pinref part="R1" gate="G$1" pin="2"/>
 <wire x1="116.84" y1="114.3" x2="116.84" y2="111.76" width="0.1524" layer="91"/>
 <junction x="116.84" y="114.3"/>
